Commit message: second commit

File: simulation/urdf/hermes.xacro (robot description, xacro)
@@ -188,8 +188,30 @@
   </link>
   <joint name="lidar_joint" type="fixed">
-    <origin xyz="0.630975 0 -0.1807467" rpy="0 0 0" />
+    <origin xyz="0.630975 0 0.4" rpy="0 0 0" />
     <parent link="base_link" />
     <child link="lidar_link" />
   </joint>
+  <gazebo>
+    <plugin name="differential_drive_controller" filename="libgazebo_ros_diff_drive.so">
+      <leftJoint>left_wheel_joint</leftJoint>
+      <odometryTopic>odom</odometryTopic>
+      <odometryFrame>odom</odometryFrame>
+      <publishWheelTF>false</publishWheelTF>
+      <publishOdomTF>true</publishOdomTF>
+      <wheelTorque>5</wheelTorque>
+      <wheelAcceleration>0</wheelAcceleration>
+      <updateRate>100</updateRate>
+      <odometrySource>world</odometrySource> <!-- 'encoder' instead of 'world' is also possible -->
+      <publishTf>1</publishTf>
+      <rosDebugLevel>na</rosDebugLevel>
+      <rightJoint>right_wheel_joint</rightJoint>
+      <robotBaseFrame>base_link</robotBaseFrame>
+      <wheelSeparation>0.25</wheelSeparation>
+      <wheelDiameter>0.07</wheelDiameter>
+      <publishWheelJointState>true</publishWheelJointState>
+      <commandTopic>cmd_vel</commandTopic>
+      <robotBaseFrame>base_link</robotBaseFrame>
+    </plugin>
+  </gazebo>
 <gazebo reference="lidar_link">
 <sensor type="ray" name="lidar_link">
@@ -206,5 +228,5 @@
               </horizontal>
               <vertical>
-                <samples>16</samples>
+                <samples>32</samples>
                 <resolution>1</resolution>
                 <min_angle>-0.25</min_angle>
